File: circuits/schematics/FSOCom.kicad_sch (KiCad schematic)
At the start: 59 parts, among them IC1 LCMXO3LF-1300E-5UWG36ITR, IC2 OPA695IDBVR, IC3 ADC08200CIMT_NOPB, J1 RJ45, Q1 IRLML2030TRPBF, U1 DP83848C, X1 ECS-2520MVQ-500-BN

Commit message: Reorganized circuit schematics, started power source design
Parts:
- removed C1: 1000pF, 2kV, symbol Device:C
- removed C10: PLACEHOLDER, symbol Device:C
- removed C11, C12, C15, C2, C3, C4, C5, C6, C7, C9: 0.1μF, symbol Device:C
- removed C13, C14, C8: 10μF, symbol Device:C
- removed C16, C17: 1μF, symbol Device:C
- removed D1, D2, D3: MTPD3001D3-030, MTPD3001D3030, symbol MTPD3001D3-030:MTPD3001D3-030
- removed IC2: OPA695IDBVR, SOT95P280X145-6N, symbol OPA695IDBVR:OPA695IDBVR
- removed IC3: ADC08200CIMT_NOPB, SOP65P640X120-24N, symbol ADC08200CIMT_NOPB:ADC08200CIMT_NOPB
- removed J1: RJ45, symbol Connector:RJ45
- removed LD1: OPV300, symbol Device:D_Laser_1C2A
- removed Q1: IRLML2030TRPBF, SOT95P237X112-3N, symbol IRLML2030TRPBF:IRLML2030TRPBF
- removed R1, R2, R3, R4: 75, symbol Device:R
- removed R10, R12, R13, R14, R19, R20, R23, R24, R25, R26, R27, R28, R9: 2.2k, symbol Device:R
- removed R11: 4.87k 1%, symbol Device:R
- removed R15, R16: PLACEHOLDER, symbol Device:R
- removed R17: 1.1k, symbol Device:R
- removed R18: 1.5k, symbol Device:R
- removed R21: 10k, symbol Device:R
- removed R22: 1k, symbol Device:R
- removed R29: 100, symbol Device:R
- removed R30: 50, symbol Device:R
- removed R5, R6, R7, R8: 49.9, symbol Device:R
- removed TR1: H1102, Transformer_SMD:Transformer_Ethernet_Bourns_PT61017PEL, symbol Transformer:PT61017PEL
- removed U1: DP83848C, Package_QFP:LQFP-48_7x7mm_P0.5mm, symbol Interface_Ethernet:DP83848C
- removed X1: ECS-2520MVQ-500-BN, Oscillator:Oscillator_SMD_ECS_2520MV-xxx-xx-4Pin_2.5x2.0mm, symbol Oscillator:ECS-2520MV-xxx-xx
Connections:
- net Laser Driver: now reaches IC1.E5 (PB4C)
- net ADC7: now reaches IC1.B3 (PT12B)
- net ADC6: now reaches IC1.B2 (PT15C)
- net ADC5: now reaches IC1.B1 (PT17C)
- net ADC4: now reaches IC1.A6 (PT9A)
- net ADC3: now reaches IC1.A5 (PT10D)
- net ADC2: now reaches IC1.A4 (PT12A)
- net ADC1: now reaches IC1.A2 (PT15D)
- net ADC0: now reaches IC1.A1 (PT17D)
- net ADCCLK: now reaches IC1.B6 (PL2D)
- net PHYTXEN: now reaches IC1.D4 (PT10A)
- net PHYCLK: now reaches IC1.E6 (PL9B)
- net PHYTX0: now reaches IC1.D2 (PT12C)
- net PHYRXDV: now reaches IC1.E3 (PB9A)
- net PHYTX1: now reaches IC1.D3 (PT11C)
- net PHYCRS: now reaches IC1.E4 (PB6D)
- net PHYRX0: now reaches IC1.E1 (PB20C)
- net PHYRX1: now reaches IC1.E2 (PB11A)
- no-connect marks 0 -> 11
Other:
- added sheet laser-driver (laser-driver.kicad_sch)
- added sheet photodiode-array (photodiode-array.kicad_sch)
- added sheet phy-interface (phy-interface.kicad_sch)
- added sheet power (power.kicad_sch)
- moved on the sheet: IC1
